File: LFO - MFOS/_autosave-LFO - MFOS.sch (KiCad schematic (older format))
At the start: 104 parts, among them J1 CFV, J10 PWXY, J11 PWC, J12 SIN, J13 PW10, J14 PW90, J15 SQR, J16 LEDA, J2 CV1, J3 CV2, J4 CV3, J5 CFL, J6 FFV, J7 TRI, J8 RMP, J9 SAW, Q1 Q_NJFET_DSG, Q2 Q_NJFET_DSG, Q3 2N3904, Q4 2N3904, Q5 2N3906, Q6 2N3904, U1 LM13700, U2 TL082, U3 TL082, U4 TL072, U5 TL082, U6 TL082

Commit message: placed components in general location on pcb uwu
Parts:
- added J17: +12V_Conn, Connector_Wire:SolderWirePad_1x02_P3.81mm_Drill1mm, symbol Connector:Conn_01x02_Female
- added J18: GND_Conn, Connector_Wire:SolderWirePad_1x02_P3.81mm_Drill1mm, symbol Connector:Conn_01x02_Female
- added J19: -12V_Conn, Connector_Wire:SolderWirePad_1x02_P3.81mm_Drill1mm, symbol Connector:Conn_01x02_Female
- C10, C5, C6, C7, C8, C9: footprint Capacitor_THT:CP_Radial_D4.0mm_P2.00mm -> Capacitor_THT:C_Rect_L7.0mm_W2.5mm_P5.00mm
Connections:
- net +12V: now also J17.1 (Pin_1), J17.2 (Pin_2)
- net -12V: now also J19.1 (Pin_1), J19.2 (Pin_2)
- net Earth: now also J18.1 (Pin_1), J18.2 (Pin_2)
Changed lines of the file:
@@
 F 0 "C5" H 8465 1146 50  0000 L CNN
 F 1 "0.1uF" H 8465 1055 50  0000 L CNN
-F 2 "Capacitor_THT:CP_Radial_D4.0mm_P2.00mm" H 8350 1100 50  0001 C CNN
+F 2 "Capacitor_THT:C_Rect_L7.0mm_W2.5mm_P5.00mm" H 8350 1100 50  0001 C CNN
 F 3 "~" H 8350 1100 50  0001 C CNN
 	1    8350 1100
@@
 F 0 "C7" H 8965 1146 50  0000 L CNN
 F 1 "0.1uF" H 8965 1055 50  0000 L CNN
-F 2 "Capacitor_THT:CP_Radial_D4.0mm_P2.00mm" H 8850 1100 50  0001 C CNN
+F 2 "Capacitor_THT:C_Rect_L7.0mm_W2.5mm_P5.00mm" H 8850 1100 50  0001 C CNN
 F 3 "~" H 8850 1100 50  0001 C CNN
 	1    8850 1100
@@
 F 0 "C9" H 9415 1146 50  0000 L CNN
 F 1 "0.1uF" H 9415 1055 50  0000 L CNN
-F 2 "Capacitor_THT:CP_Radial_D4.0mm_P2.00mm" H 9300 1100 50  0001 C CNN
+F 2 "Capacitor_THT:C_Rect_L7.0mm_W2.5mm_P5.00mm" H 9300 1100 50  0001 C CNN
 F 3 "~" H 9300 1100 50  0001 C CNN
 	1    9300 1100
@@
 F 0 "C6" H 8465 1696 50  0000 L CNN
 F 1 "0.1uF" H 8465 1605 50  0000 L CNN
-F 2 "Capacitor_THT:CP_Radial_D4.0mm_P2.00mm" H 8350 1650 50  0001 C CNN
+F 2 "Capacitor_THT:C_Rect_L7.0mm_W2.5mm_P5.00mm" H 8350 1650 50  0001 C CNN
 F 3 "~" H 8350 1650 50  0001 C CNN
 	1    8350 1650
@@
 F 0 "C8" H 8965 1696 50  0000 L CNN
 F 1 "0.1uF" H 8965 1605 50  0000 L CNN
-F 2 "Capacitor_THT:CP_Radial_D4.0mm_P2.00mm" H 8850 1650 50  0001 C CNN
+F 2 "Capacitor_THT:C_Rect_L7.0mm_W2.5mm_P5.00mm" H 8850 1650 50  0001 C CNN
 F 3 "~" H 8850 1650 50  0001 C CNN
 	1    8850 1650
@@
 F 0 "C10" H 9415 1696 50  0000 L CNN
 F 1 "0.1uF" H 9415 1605 50  0000 L CNN
-F 2 "Capacitor_THT:CP_Radial_D4.0mm_P2.00mm" H 9300 1650 50  0001 C CNN
+F 2 "Capacitor_THT:C_Rect_L7.0mm_W2.5mm_P5.00mm" H 9300 1650 50  0001 C CNN
 F 3 "~" H 9300 1650 50  0001 C CNN
 	1    9300 1650
@@
 $EndComp
 Connection ~ 9950 3400
+$Comp
+L Connector:Conn_01x02_Female J17
+U 1 1 60223451
+P 7850 650
+F 0 "J17" V 7788 462 50  0000 R CNN
+F 1 "+12V_Conn" V 7697 462 50  0000 R CNN
+F 2 "Connector_Wire:SolderWirePad_1x02_P3.81mm_Drill1mm" H 7850 650 50  0001 C CNN
+F 3 "~" H 7850 650 50  0001 C CNN
+	1    7850 650
+	0    -1   -1   0
+$EndComp
+$Comp
+L Connector:Conn_01x02_Female J18
+U 1 1 60224A8B
+P 7850 1150
+F 0 "J18" V 7788 962 50  0000 R CNN
+F 1 "GND_Conn" V 7697 962 50  0000 R CNN
+F 2 "Connector_Wire:SolderWirePad_1x02_P3.81mm_Drill1mm" H 7850 1150 50  0001 C CNN
+F 3 "~" H 7850 1150 50  0001 C CNN
+	1    7850 1150
+	0    -1   -1   0
+$EndComp
+$Comp
+L Connector:Conn_01x02_Female J19
+U 1 1 60225244
+P 7850 1700
+F 0 "J19" V 7788 1512 50  0000 R CNN
+F 1 "-12V_Conn" V 7697 1512 50  0000 R CNN
+F 2 "Connector_Wire:SolderWirePad_1x02_P3.81mm_Drill1mm" H 7850 1700 50  0001 C CNN
+F 3 "~" H 7850 1700 50  0001 C CNN
+	1    7850 1700
+	0    -1   -1   0
+$EndComp
+Wire Wire Line
+	8200 850  7950 850
+Connection ~ 8200 850
+Wire Wire Line
+	7850 850  7950 850
+Connection ~ 7950 850
+Wire Wire Line
+	7850 1350 7950 1350
+Wire Wire Line
+	8200 1350 7950 1350
+Connection ~ 8200 1350
+Connection ~ 7950 1350
+Wire Wire Line
+	7850 1900 7950 1900
+Wire Wire Line
+	7950 1900 8200 1900
+Connection ~ 7950 1900
+Connection ~ 8200 1900
 $EndSCHEMATC
