File: Dual Universal Slope Generator - CGS/Dual Universal Slope Generator - CGS.sch (KiCad schematic (older format))
At the start: 81 parts, among them J1 CV_IN_A, J17 CV_POT_A, J18 FALL_POT_A, J19 RISE_POT_A, J2 TRIG_IN_A, J20 SW_RISE_A, J21 SW_FALL_A, J27 LED_A, J3 IN_A, J4 1V/OCT_A, J5 DC_OUT_A, J6 AC_COUPLED_OUT_A, J7 END_OUT_A, J8 BIPOLAR_OUT_A, Q1 2N3904, Q2 2N3906, Q3 2N3906, Q4 2N3906, Q5 2N3904, Q6 BC547, SW1 SW_SPDT_MSM, U1 LF353, U2 TL072, U3 LM3900

Commit message: lots of stuff tbh
Other:
- note added: "LED and driver deadbugged (not on PCB)\n"
Changed lines of the file:
@@
 	1    0    0    -1
 $EndComp
+Text Notes 7100 5700 0    50   ~ 0
+LED and driver deadbugged (not on PCB)\n
 $EndSCHEMATC
