File: Totem Pole VCF -EAGLE/totem_pole_vcf.brd (EAGLE design)
At the start: 160 x 100 mm, 98 parts, among them IC1 LF412N, IC2 TL074P, J1 PWR_CON, Q1 2N3819, T1 2SA1015, T2 2SC1815, T3 2SC1815, T4 2SC1815, T5 2SC1815, T6 2SC1815

Commit message: fixed eagle gerbers
Other:
- board size 160 x 100 mm -> 86 x 88 mm
Changed lines of the file:
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@@
 <board>
 <plain>
-<wire x1="0" y1="0" x2="160" y2="0" width="0" layer="20"/>
-<wire x1="160" y1="0" x2="160" y2="100" width="0" layer="20"/>
-<wire x1="160" y1="100" x2="0" y2="100" width="0" layer="20"/>
-<wire x1="0" y1="100" x2="0" y2="0" width="0" layer="20"/>
+<wire x1="-0.00394375" y1="11.9975875" x2="86.0006875" y2="11.99796875" width="0" layer="20"/>
+<wire x1="86.0006875" y1="11.99796875" x2="86.003259375" y2="100.0039875" width="0" layer="20"/>
+<wire x1="86.003259375" y1="100.0039875" x2="0.00018125" y2="99.998515625" width="0" layer="20"/>
+<wire x1="0.00018125" y1="99.998515625" x2="-0.00394375" y2="11.9975875" width="0" layer="20"/>
 <wire x1="0" y1="100" x2="86" y2="100" width="0.1524" layer="46"/>
 <wire x1="86" y1="12" x2="0" y2="12" width="0.1524" layer="46"/>
