File: Sequencer - MFOS/Analog.sch (KiCad schematic (older format))
At the start: 127 parts, among them J27 CV1_GL, J28 CV2_GL, J29 CV3, J30 CV4, J31 7C, J32 7F, J33 6C, J34 6F, J35 5C, J36 5F, J37 4C, J38 4F, J39 3C, J40 3F, J41 2C, J42 2F, J43 1C, J44 1F, J45 0C, J46 0F, J47 12C, J48 12F, J49 13C, J50 13F, J51 14C, J52 14F, J53 15C, J54 15F, J55 8C, J56 8F, J57 9C, J58 9F, J59 10C, J60 10F, J61 11C, J62 11F, J70 PORT1W, J71 PORT3, J72 VSRC, U10 TL082, U11 CD74HC4067M, U9 TL084

Commit message: checked over sequencer schematic
Parts:
- R37: value 10k? -> 10k
- R86, R87, R88, R89: value R_US -> 1k
Connections:
- net Earth: now also R48.1; no longer R48.2
- net at C27.2, R49.2, U9.2 (-): now also R48.2; no longer R48.1
Other:
- moved on the sheet: C25, D49, R37, R38, R48
Changed lines of the file:
@@
 L Device:R_US R48
 U 1 1 612A5A47
-P 1250 1850
-F 0 "R48" V 1450 1850 50  0000 C CNN
-F 1 "100k" V 1350 1850 50  0000 C CNN
-F 2 "" V 1290 1840 50  0001 C CNN
-F 3 "~" H 1250 1850 50  0001 C CNN
-	1    1250 1850
-	0    1    1    0
-$EndComp
-Wire Wire Line
-	1450 1850 1400 1850
+P 1300 2000
+F 0 "R48" V 1500 2000 50  0000 C CNN
+F 1 "100k" V 1400 2000 50  0000 C CNN
+F 2 "" V 1340 1990 50  0001 C CNN
+F 3 "~" H 1300 2000 50  0001 C CNN
+	1    1300 2000
+	-1   0    0    1
+$EndComp
 Connection ~ 1450 1850
 Wire Wire Line
@@
 L power:Earth #PWR051
 U 1 1 612EBAB1
-P 950 2000
-F 0 "#PWR051" H 950 1750 50  0001 C CNN
-F 1 "Earth" H 950 1850 50  0001 C CNN
-F 2 "" H 950 2000 50  0001 C CNN
-F 3 "~" H 950 2000 50  0001 C CNN
-	1    950  2000
-	1    0    0    -1
-$EndComp
-Wire Wire Line
-	1100 1900 1100 1850
+P 1000 2150
+F 0 "#PWR051" H 1000 1900 50  0001 C CNN
+F 1 "Earth" H 1000 2000 50  0001 C CNN
+F 2 "" H 1000 2150 50  0001 C CNN
+F 3 "~" H 1000 2150 50  0001 C CNN
+	1    1000 2150
+	1    0    0    -1
+$EndComp
 $Comp
 L Device:C C25
 U 1 1 6130F6EB
-P 950 1750
-F 0 "C25" V 1200 1750 50  0000 C CNN
-F 1 "0.1u" V 1100 1750 50  0000 C CNN
-F 2 "" H 988 1600 50  0001 C CNN
-F 3 "~" H 950 1750 50  0001 C CNN
-	1    950  1750
+P 1000 1800
+F 0 "C25" V 1250 1800 50  0000 C CNN
+F 1 "0.1u" V 1150 1800 50  0000 C CNN
+F 2 "" H 1038 1650 50  0001 C CNN
+F 3 "~" H 1000 1800 50  0001 C CNN
+	1    1000 1800
 	-1   0    0    1
 $EndComp
-Wire Wire Line
-	1100 1900 950  1900
-Wire Wire Line
-	1100 1650 1100 1600
-Wire Wire Line
-	1100 1600 1000 1600
 $Comp
 L Device:D_Zener D49
 U 1 1 6135A66D
-P 800 1250
-F 0 "D49" H 900 1050 50  0000 C CNN
-F 1 "D_Zener" H 800 1125 50  0000 C CNN
-F 2 "" H 800 1250 50  0001 C CNN
-F 3 "~" H 800 1250 50  0001 C CNN
-	1    800  1250
+P 800 1300
+F 0 "D49" H 900 1100 50  0000 C CNN
+F 1 "D_Zener" H 800 1175 50  0000 C CNN
+F 2 "" H 800 1300 50  0001 C CNN
+F 3 "~" H 800 1300 50  0001 C CNN
+	1    800  1300
 	-1   0    0    1
 $EndComp
@@
 L power:Earth #PWR050
 U 1 1 6135C65F
-P 600 1300
-F 0 "#PWR050" H 600 1050 50  0001 C CNN
-F 1 "Earth" H 600 1150 50  0001 C CNN
-F 2 "" H 600 1300 50  0001 C CNN
-F 3 "~" H 600 1300 50  0001 C CNN
-	1    600  1300
-	1    0    0    -1
-$EndComp
-Wire Wire Line
-	600  1300 600  1250
-Wire Wire Line
-	600  1250 650  1250
+P 600 1350
+F 0 "#PWR050" H 600 1100 50  0001 C CNN
+F 1 "Earth" H 600 1200 50  0001 C CNN
+F 2 "" H 600 1350 50  0001 C CNN
+F 3 "~" H 600 1350 50  0001 C CNN
+	1    600  1350
+	1    0    0    -1
+$EndComp
+Wire Wire Line
+	600  1350 600  1300
+Wire Wire Line
+	600  1300 650  1300
 $Comp
 L Device:R_US R37
 U 1 1 6138302C
-P 1000 1050
-F 0 "R37" H 850 1000 50  0000 C CNN
-F 1 "10k?" H 850 1100 50  0000 C CNN
-F 2 "" V 1040 1040 50  0001 C CNN
-F 3 "~" H 1000 1050 50  0001 C CNN
-	1    1000 1050
+P 1000 1100
+F 0 "R37" H 850 1050 50  0000 C CNN
+F 1 "10k" H 850 1150 50  0000 C CNN
+F 2 "" V 1040 1090 50  0001 C CNN
+F 3 "~" H 1000 1100 50  0001 C CNN
+	1    1000 1100
 	-1   0    0    1
 $EndComp
@@
 L power:+12V #PWR052
 U 1 1 61386B95
-P 1000 850
-F 0 "#PWR052" H 1000 700 50  0001 C CNN
-F 1 "+12V" H 1015 1023 50  0000 C CNN
-F 2 "" H 1000 850 50  0001 C CNN
-F 3 "" H 1000 850 50  0001 C CNN
-	1    1000 850
-	1    0    0    -1
-$EndComp
-Wire Wire Line
-	1000 850  1000 900
-Wire Wire Line
-	950  1250 1000 1250
-Wire Wire Line
-	1000 1250 1000 1200
+P 1000 900
+F 0 "#PWR052" H 1000 750 50  0001 C CNN
+F 1 "+12V" H 1015 1073 50  0000 C CNN
+F 2 "" H 1000 900 50  0001 C CNN
+F 3 "" H 1000 900 50  0001 C CNN
+	1    1000 900
+	1    0    0    -1
+$EndComp
+Wire Wire Line
+	1000 900  1000 950
+Wire Wire Line
+	950  1300 1000 1300
+Wire Wire Line
+	1000 1300 1000 1250
 $Comp
 L Device:R_US R38
 U 1 1 613D1236
-P 1000 1450
-F 0 "R38" H 1100 1400 50  0000 C CNN
-F 1 "47k" H 1150 1500 50  0000 C CNN
-F 2 "" V 1040 1440 50  0001 C CNN
-F 3 "~" H 1000 1450 50  0001 C CNN
-	1    1000 1450
+P 1000 1500
+F 0 "R38" H 1100 1450 50  0000 C CNN
+F 1 "47k" H 1150 1550 50  0000 C CNN
+F 2 "" V 1040 1490 50  0001 C CNN
+F 3 "~" H 1000 1500 50  0001 C CNN
+	1    1000 1500
 	-1   0    0    1
 $EndComp
-Connection ~ 1000 1600
-Wire Wire Line
-	1000 1600 950  1600
-Wire Wire Line
-	1000 1300 1000 1250
-Connection ~ 1000 1250
-Wire Wire Line
-	950  2000 950  1900
-Connection ~ 950  1900
+Wire Wire Line
+	1000 1350 1000 1300
+Connection ~ 1000 1300
 Wire Wire Line
 	2150 1750 2300 1750
@@
 P 2200 5100
 F 0 "R86" V 1995 5100 50  0000 C CNN
-F 1 "R_US" V 2086 5100 50  0000 C CNN
+F 1 "1k" V 2086 5100 50  0000 C CNN
 F 2 "" V 2240 5090 50  0001 C CNN
 F 3 "~" H 2200 5100 50  0001 C CNN
@@
 P 2200 5250
 F 0 "R87" V 2400 5250 50  0000 C CNN
-F 1 "R_US" V 2300 5250 50  0000 C CNN
+F 1 "1k" V 2300 5250 50  0000 C CNN
 F 2 "" V 2240 5240 50  0001 C CNN
 F 3 "~" H 2200 5250 50  0001 C CNN
@@
 P 2200 6100
 F 0 "R88" V 1995 6100 50  0000 C CNN
-F 1 "R_US" V 2086 6100 50  0000 C CNN
+F 1 "1k" V 2086 6100 50  0000 C CNN
 F 2 "" V 2240 6090 50  0001 C CNN
 F 3 "~" H 2200 6100 50  0001 C CNN
@@
 P 2200 6850
 F 0 "R89" V 1995 6850 50  0000 C CNN
-F 1 "R_US" V 2086 6850 50  0000 C CNN
+F 1 "1k" V 2086 6850 50  0000 C CNN
 F 2 "" V 2240 6840 50  0001 C CNN
 F 3 "~" H 2200 6850 50  0001 C CNN
@@
 $EndComp
 Connection ~ 700  4900
+$Comp
+L power:Earth #PWR?
+U 1 1 61DE3A9B
+P 1300 2150
+F 0 "#PWR?" H 1300 1900 50  0001 C CNN
+F 1 "Earth" H 1300 2000 50  0001 C CNN
+F 2 "" H 1300 2150 50  0001 C CNN
+F 3 "~" H 1300 2150 50  0001 C CNN
+	1    1300 2150
+	1    0    0    -1
+$EndComp
+Wire Wire Line
+	1300 1850 1450 1850
+Wire Wire Line
+	1100 1650 1000 1650
+Connection ~ 1000 1650
+Wire Wire Line
+	1000 1950 1000 2150
 $EndSCHEMATC

Commit message: sequencer pcb designed and base silkscreen
Parts:
- C25, C26, C27, C30: footprint (none) -> Capacitor_THT:C_Rect_L7.0mm_W2.5mm_P5.00mm
- C28, C29: footprint (none) -> Capacitor_THT:CP_Radial_D4.0mm_P2.00mm
- D49: footprint (none) -> Diode_THT:D_T-1_P5.08mm_Horizontal
- J27, J28, J29, J30, J31, J32, J33, J34, J35, J36, J37, J38, J39, J40, J41, J42, J43, J44, J45, J46, J47, J48, J49, J50, J51, J52, J53, J54, J55, J56, J57, J58, J59, J60, J61, J62, J70, J71, J72: footprint (none) -> Connector_Wire:SolderWirePad_1x01_Drill1mm
- R37, R38, R39, R48, R49, R50, R51, R52, R53, R54, R55, R56, R57, R58, R59, R60, R61, R62, R63, R64, R65, R66, R67, R68, R69, R70, R71, R72, R73, R74, R75, R76, R77, R78, R79, R80, R81, R82, R83, R84, R85, R86, R87, R88, R89: footprint (none) -> Resistor_THT:R_Axial_DIN0207_L6.3mm_D2.5mm_P7.62mm_Horizontal
- U10: footprint (none) -> Package_DIP:DIP-8_W7.62mm_Socket
- U11: footprint Package_SO:SOIC-24W_7.5x15.4mm_P1.27mm -> Package_DIP:DIP-24_W15.24mm_Socket
- U9: footprint (none) -> Package_DIP:DIP-14_W7.62mm_Socket
