File: Sequencer - MFOS/Sequencer - MFOS.kicad_pcb (KiCad board)
At the start: 2 copper layers, 176.3 x 101.6 mm, 222 parts, among them J1 STUP, J10 S7, J11 S6, J12 S5, J13 S4, J14 S3, J15 S2, J16 S1, J17 S0, J18 S8, J19 S9, J2 STDN, J20 S10, J21 S11, J22 RIN, J23 S12, J24 S13, J25 S14, J26 S15, J27 CV1_GL, J28 CV2_GL, J29 CV3, J3 XSTP, J30 CV4, J31 7C, J32 7F, J33 6C, J34 6F, J35 5C, J36 5F, J37 4C, J38 4F, J39 3C, J4 XCLK, J40 3F, J41 2C, J42 2F, J43 1C, J44 1F, J45 0C, J46 0F, J47 12C, J48 12F, J49 13C, J5 CKOUT, J50 13F, J51 14C, J52 14F, J53 15C, J54 15F, J55 8C, J56 8F, J57 9C, J58 9F, J59 10C, J6 GATE, J60 10F, J61 11C, J62 11F, J63 CK_RT1W, J64 CK_RT3, J65 STRN, J66 REV, J67 STP, J68 RESET, J69 RAND, J7 TRIG, J70 PORT1W, J71 PORT3, J72 VSRC, J73 +12V_Conn, J74 GND_Conn, J75 -12V_Conn, J8 GB, J9 CBUS, Q1 2N3904, U1 40106, U10 TL082, U11 CD74HC4067M, U12 CD4094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

Commit message: made silkscreens pretty
Routing:
- added copper zone on B.Cu, net Earth
- added copper zone on F.Cu, net Earth

Commit message: uwu
Other:
- board text added: "MFOS"
Changed lines of the file:
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@@
   (general
     (thickness 1.6)
-    (drawings 994)
+    (drawings 995)
     (tracks 1393)
     (zones 0)
@@
     )
   )
+  (gr_text MFOS (at 36.3474 93.4466) (layer F.SilkS)
+    (effects (font (size 1.5 1.5) (thickness 0.3)))
+  )
   (gr_circle (center 41.275 29.083) (end 41.6814 31.4452) (layer F.SilkS) (width 0.3))

Commit message: literally so much stuff
Changed lines of the file:
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@@
     (47 F.CrtYd user hide)
     (48 B.Fab user hide)
-    (49 F.Fab user hide)
+    (49 F.Fab user)
   )
   (setup
@@
     (effects (font (size 1 1) (thickness 0.15)))
   )
-  (gr_text F (at 77.1144 33.5026) (layer F.SilkS)
+  (gr_text F (at 72.1106 34.0868) (layer F.SilkS)
     (effects (font (size 1 1) (thickness 0.15)))
   )
-  (gr_text C (at 73.3298 33.655) (layer F.SilkS)
+  (gr_text C (at 77.3176 33.4772) (layer F.SilkS)
     (effects (font (size 1 1) (thickness 0.15)))
   )
@@
     (effects (font (size 1 1) (thickness 0.15)))
   )
-  (gr_text F (at 66.9798 34.7726) (layer F.SilkS)
+  (gr_text F (at 62.2808 36.322) (layer F.SilkS)
     (effects (font (size 1 1) (thickness 0.15)))
   )
-  (gr_text C (at 62.0776 36.2458) (layer F.SilkS)
+  (gr_text C (at 66.5734 34.8488) (layer F.SilkS)
     (effects (font (size 1 1) (thickness 0.15)))
   )
