File: Sequencer - MFOS/Dual Micro Sample Hold - MFOS/Dual Micro Sample Hold - MFOS.kicad_pcb (KiCad board)
At the start: 2 copper layers, 58.2 x 46.7 mm, 44 parts, among them J1 +12V_Conn, J10 TRIG_A, J11 CV_OUT_A, J12 GLIDE_OUT_A, J2 GND_Conn, J3 -12V_Conn, J4 IN_A, J5 SampRate_1W_A, J6 SampRate_3_A, J7 LED_A, J8 Glide_1W_A, J9 Glide_3_A, Q1 Q_NJFET_DSG, U1 LF444

Commit message: made silkscreens pretty
Routing:
- added copper zone on B.Cu, net Earth
- added copper zone on F.Cu, net Earth
