File: Ambisonics/B_Format_Mic_Encoder/B_Format_Mic_Encoder.sch (KiCad schematic (older format))
At the start: 104 parts, among them J1 A_Format_In, J2 B_Form_Out, J3 B_Form_Out, J4 PWR_OUT, J5 PWR_IN, Q1 2N4403, Q2 2N4403, Q3 2N4403, Q4 2N4403, Q5 2N4403, Q6 2N4403, Q7 2N4403, Q8 2N4403, U1 TL074, U2 TL074

Commit message: ambisonic pcbsdoneee
Parts:
- C17, C18: footprint Capacitor_THT:C_Rect_L7.0mm_W2.5mm_P5.00mm -> Capacitor_THT:CP_Radial_D6.3mm_P2.50mm
Changed lines of the file:
@@
 F 0 "C18" H 10265 1496 50  0000 L CNN
 F 1 "22u" H 10265 1405 50  0000 L CNN
-F 2 "Capacitor_THT:C_Rect_L7.0mm_W2.5mm_P5.00mm" H 10150 1450 50  0001 C CNN
+F 2 "Capacitor_THT:CP_Radial_D6.3mm_P2.50mm" H 10150 1450 50  0001 C CNN
 F 3 "~" H 10150 1450 50  0001 C CNN
 	1    10150 1450
@@
 F 0 "C17" H 10265 1096 50  0000 L CNN
 F 1 "22u" H 10265 1005 50  0000 L CNN
-F 2 "Capacitor_THT:C_Rect_L7.0mm_W2.5mm_P5.00mm" H 10150 1050 50  0001 C CNN
+F 2 "Capacitor_THT:CP_Radial_D6.3mm_P2.50mm" H 10150 1050 50  0001 C CNN
 F 3 "~" H 10150 1050 50  0001 C CNN
 	1    10150 1050
