File: Voltage Quantizer - MFOS/Voltage Quantizer - MFOS.sch (KiCad schematic (older format))
At the start: 83 parts, among them J1 S1C, J10 Vin_3, J11 +12V, J12 GND, J13 -12V, J2 S2C, J3 S1A, J4 S1B, J5 S2A, J6 S2B, J7 Vout, J8 Vin_1, J9 Vin_2, SW1 SW_SPDT, SW2 SW_SPDT, U1 40106, U2 40193, U3 40193, U4 TL084, U5 TL071, U6 4013, U7 4042

Commit message: hii
Parts:
- gave numbers to parts that had none: 1
Changed lines of the file:
@@
 	10400 1550 10400 1650
 $Comp
-L Connector:Conn_01x01_Female J?
+L Connector:Conn_01x01_Female J14
 U 1 1 6102E865
 P 10750 4300
-F 0 "J?" H 10778 4326 50  0000 L CNN
+F 0 "J14" H 10778 4326 50  0000 L CNN
 F 1 "Vadj" H 10778 4235 50  0000 L CNN
 F 2 "Connector_Wire:SolderWirePad_1x01_Drill1mm" H 10750 4300 50  0001 C CNN
