File: Voltage Quantizer - MFOS/Voltage Quantizer - MFOS.kicad_pcb (KiCad board)
At the start: 2 copper layers, 88.1 x 87.4 mm, 84 parts, among them J1 S1C, J10 Vin_3, J11 +12V, J12 GND, J13 -12V, J14 Vadj, J2 S2C, J3 S1A, J4 S1B, J5 S2A, J6 S2B, J7 Vout, J8 Vin_1, J9 Vin_2, U1 40106, U2 40193, U3 40193, U4 TL084, U5 TL071, U6 4013, U7 4042

Commit message: literally so much stuff
Routing:
- added copper zone on B.Cu, net Earth
- added copper zone on F.Cu, net Earth
