File: Analog Shift Register - CGS/Analog Shift Register - CGS.kicad_pcb (KiCad board)
At the start: 2 copper layers, 88.9 x 89.9 mm, 57 parts, among them J1 CV_In, J2 CLK_IN, J3 +12V_Conn, J4 GND_Conn, J5 -12V_Conn, J6 Out 3, J7 Out_2, J8 Out_1, U1 TL084, U2 TL071, U3 4052, U4 4024, U5 LF356, U6 LF356, U7 LF356, U8 LF356, U9 4052

Commit message: literally so much stuff
Routing:
- added copper zone on B.Cu, net Earth
- added copper zone on F.Cu, net Earth
