File: Noise Cornucopia - MFOS/Noise Cornucopia - MFOS.kicad_pcb (KiCad board)
At the start: 2 copper layers, 73.4 x 68.1 mm, 80 parts, among them J1 GRNS_3, J10 Q3, J11 Q4, J12 Q5, J13 Q6, J14 GATE_JMP, J15 White, J16 LP_White, J17 GATE_OUT, J18 HP_White, J19 LED, J2 GRNS_W1, J20 +12V_Conn, J21 GND_Conn?, J22 -12V_Conn, J3 Gate_F_W1, J4 Gate_F_3, J5 Grain, J6 Grain_HP, J7 Q0, J8 Q1, J9 Q2, Q1 2N3904, Q2 2N3904, U1 TL072, U2 TL072, U3 TL072, U4 4024, U5 TL072

Commit message: made silkscreens pretty
Routing:
- added copper zone on B.Cu, net Earth
- added copper zone on F.Cu, net Earth
