File: Triple Waveshaper - CGS/Triple Waveshaper - CGS.sch (KiCad schematic (older format))
At the start: 75 parts, among them J1 CV_1_A, J10 Sum_In_C, J11 IN_C, J12 DC_OUT_A, J13 AC_OUT_A, J14 DC_OUT_B, J15 AC_OUT_B, J16 DC_OUT_C, J17 AC_OUT_C, J18 +12V_Conn, J19 GND_Conn, J2 CV_1_B, J20 -12V_Conn, J21 AUX_In_A, J3 CV_1_C, J4 CV_2_A, J5 CV_2_B, J6 CV_2_C, J7 IN_A, J8 Sum_In_B, J9 IN_B, U1 LM3900

Commit message: added triple waveshaper pcb
Parts:
- RV1, RV2, RV3: footprint (none) -> Potentiometer_THT:Potentiometer_Runtron_RM-065_Vertical
Changed lines of the file:
@@
 EESchema Schematic File Version 4
+LIBS:Triple Waveshaper - CGS-cache
 EELAYER 29 0
 EELAYER END
@@
 F 0 "RV1" V 3037 1550 50  0000 C CNN
 F 1 "20k" V 2946 1550 50  0000 C CNN
-F 2 "" H 3150 1550 50  0001 C CNN
+F 2 "Potentiometer_THT:Potentiometer_Runtron_RM-065_Vertical" H 3150 1550 50  0001 C CNN
 F 3 "~" H 3150 1550 50  0001 C CNN
 	1    3150 1550
@@
 F 0 "RV2" V 3037 3650 50  0000 C CNN
 F 1 "20k" V 2946 3650 50  0000 C CNN
-F 2 "" H 3150 3650 50  0001 C CNN
+F 2 "Potentiometer_THT:Potentiometer_Runtron_RM-065_Vertical" H 3150 3650 50  0001 C CNN
 F 3 "~" H 3150 3650 50  0001 C CNN
 	1    3150 3650
@@
 F 0 "RV3" V 3037 5900 50  0000 C CNN
 F 1 "20k" V 2946 5900 50  0000 C CNN
-F 2 "" H 3150 5900 50  0001 C CNN
+F 2 "Potentiometer_THT:Potentiometer_Runtron_RM-065_Vertical" H 3150 5900 50  0001 C CNN
 F 3 "~" H 3150 5900 50  0001 C CNN
 	1    3150 5900

Commit message: literally so much stuff
Parts:
- R16, R17, R18: value R_US -> 1M5
- R4, R5, R6: value R_US -> 100k
Changed lines of the file:
@@
 P 1750 2600
 F 0 "R16" V 1545 2600 50  0000 C CNN
-F 1 "R_US" V 1636 2600 50  0000 C CNN
+F 1 "1M5" V 1636 2600 50  0000 C CNN
 F 2 "Resistor_THT:R_Axial_DIN0207_L6.3mm_D2.5mm_P7.62mm_Horizontal" V 1790 2590 50  0001 C CNN
 F 3 "~" H 1750 2600 50  0001 C CNN
@@
 P 1300 2750
 F 0 "R4" H 1232 2704 50  0000 R CNN
-F 1 "R_US" H 1232 2795 50  0000 R CNN
+F 1 "100k" H 1232 2795 50  0000 R CNN
 F 2 "Resistor_THT:R_Axial_DIN0207_L6.3mm_D2.5mm_P7.62mm_Horizontal" V 1340 2740 50  0001 C CNN
 F 3 "~" H 1300 2750 50  0001 C CNN
@@
 P 1750 4700
 F 0 "R17" V 1545 4700 50  0000 C CNN
-F 1 "R_US" V 1636 4700 50  0000 C CNN
+F 1 "1M5" V 1636 4700 50  0000 C CNN
 F 2 "Resistor_THT:R_Axial_DIN0207_L6.3mm_D2.5mm_P7.62mm_Horizontal" V 1790 4690 50  0001 C CNN
 F 3 "~" H 1750 4700 50  0001 C CNN
@@
 P 1300 4850
 F 0 "R5" H 1232 4804 50  0000 R CNN
-F 1 "R_US" H 1232 4895 50  0000 R CNN
+F 1 "100k" H 1232 4895 50  0000 R CNN
 F 2 "Resistor_THT:R_Axial_DIN0207_L6.3mm_D2.5mm_P7.62mm_Horizontal" V 1340 4840 50  0001 C CNN
 F 3 "~" H 1300 4850 50  0001 C CNN
@@
 P 1750 6950
 F 0 "R18" V 1545 6950 50  0000 C CNN
-F 1 "R_US" V 1636 6950 50  0000 C CNN
+F 1 "1M5" V 1636 6950 50  0000 C CNN
 F 2 "Resistor_THT:R_Axial_DIN0207_L6.3mm_D2.5mm_P7.62mm_Horizontal" V 1790 6940 50  0001 C CNN
 F 3 "~" H 1750 6950 50  0001 C CNN
@@
 P 1300 7100
 F 0 "R6" H 1232 7054 50  0000 R CNN
-F 1 "R_US" H 1232 7145 50  0000 R CNN
+F 1 "100k" H 1232 7145 50  0000 R CNN
 F 2 "Resistor_THT:R_Axial_DIN0207_L6.3mm_D2.5mm_P7.62mm_Horizontal" V 1340 7090 50  0001 C CNN
 F 3 "~" H 1300 7100 50  0001 C CNN
