File: VCF - MFOS/VCF - MFOS.kicad_pcb (KiCad board)
At the start: 2 copper layers, 127 x 101.6 mm, 108 parts, among them J1 AIN1, J10 FOUT, J11 XRES, J12 +12V, J13 GND, J14 -12V, J2 AIN2, J3 AIN3, J4 CV1, J5 CV2, J6 CV3, J7 CO3, J8 CO2, J9 C01, Q1 2N3906, Q2 2N3906, Q3 2N3906, Q4 2N3904, Q5 2N3904, Q6 2N3906, U1 TL084, U2 LM13700, U3 TL082, U4 TL082, U5 LM13700, U6 TL082, U7 LM13700, U8 TL082

Commit message: vcf done
Parts:
- moved U7 97.7 mm to (129.5, 17.7), turned to 0 degrees
- moved C5 92.6 mm to (88.1, 105.3), turned to 220 degrees
- moved R21 90.3 mm to (99.8, 105.4), turned to 130 degrees
- moved J11 86.2 mm to (72.6, 22.4), turned to 0 degrees
- moved U2 86.2 mm to (86.6, 101.5), turned to 130 degrees
- moved R17 86.1 mm to (102.7, 102.9), turned to 130 degrees
- moved R54 85.7 mm to (117.1, 18.6), turned to 0 degrees
- moved R31 84.9 mm to (110.2, 100.0), turned to 130 degrees
- moved R19 84.7 mm to (92.1, 101.9), turned to 310 degrees
- moved R44 82.1 mm to (76.4, 22.4), turned to 0 degrees
- moved R20 81.6 mm to (116.9, 96.1), turned to 130 degrees
- moved R55 81.1 mm to (124.7, 26.2), turned to 270 degrees
- moved R48 80.8 mm to (86.6, 18.6), turned to 0 degrees
- moved R40 80.3 mm to (119.8, 93.6), turned to 130 degrees
- moved R52 79.3 mm to (106.9, 18.6), turned to 0 degrees
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Routing:
- net Earth: track 256.2 -> 137.2 mm, vias 0 -> 2
- net +12V: track 35.7 -> 137.2 mm, vias 3 -> 8
- net -12V: track 368.1 -> 436.6 mm
- net RA: track 43.2 -> 99.3 mm
- net Net-(C6-Pad2): track 89.0 -> 36.9 mm, vias 1 -> 0
- net Net-(Q4-Pad1): track 30.0 -> 55.8 mm
- net Net-(C8-Pad1): track 27.6 -> 53.2 mm
- net Net-(R38-Pad2): track 105.0 -> 83.9 mm, vias 0 -> 2
- net Net-(C7-Pad1): track 45.2 -> 66.1 mm
- net Net-(C9-Pad1): track 45.7 -> 27.9 mm
- net RB: track 146.1 -> 132.0 mm
- net Net-(C4-Pad1): track 45.7 -> 59.0 mm, vias 0 -> 1
- net Net-(R58-Pad1): track 17.5 -> 29.7 mm
- net Net-(R53-Pad2): track 5.08 -> 8.21 mm
- net Net-(R12-Pad1): track 21.7 -> 24.7 mm
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Other:
- rule pad_to_mask_clearance: 0 -> 0.051
- rule via_min_size: 0.4 -> 0.6
- board text added: "+12V"
- board text added: "-12V"
- board text added: "AIN1"
- board text added: "AIN2"
- board text added: "AIN3"
- board text added: "CO1"
- board text added: "CO2"
- board text added: "CO3"
- board text added: "CV1"
- board text added: "CV2"
- board text added: "CV3"
- board text added: "Earth"
- board text added: "FOUT"
- board text added: "RES1"
- board text added: "RES2"
- board text added: "RES3"
- board text added: "XRES"

Commit message: front panel work
Parts:
- added REF**: MountingHole_3.5mm, MountingHole:MountingHole_3.5mm, F.Cu at (18.3, 108.7)
- added REF**: MountingHole_3.5mm, MountingHole:MountingHole_3.5mm, F.Cu at (18.3, 18.3)
Changed lines of the file:
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@@
     (tracks 475)
     (zones 0)
-    (modules 108)
+    (modules 110)
     (nets 84)
   )
@@
     (add_net RB)
   )
+  (module MountingHole:MountingHole_3.5mm (layer F.Cu)
+    (at 18.288 108.712)
+    (descr "Mounting Hole 3.5mm, no annular")
+    (tags "mounting hole 3.5mm no annular")
+    (attr virtual)
+    (fp_text reference REF** (at 0 -4.5) (layer F.SilkS)
+      (effects (font (size 1 1) (thickness 0.15)))
+    )
+    (fp_text value MountingHole_3.5mm (at 0 4.5) (layer F.Fab)
+      (effects (font (size 1 1) (thickness 0.15)))
+    )
+    (fp_circle (center 0 0) (end 3.75 0) (layer F.CrtYd) (width 0.05))
+    (fp_circle (center 0 0) (end 3.5 0) (layer Cmts.User) (width 0.15))
+    (fp_text user %R (at 0.3 0) (layer F.Fab)
+      (effects (font (size 1 1) (thickness 0.15)))
+    )
+    (pad 1 np_thru_hole circle (at 0 0) (size 3.5 3.5) (drill 3.5) (layers *.Cu *.Mask))
+  )
+  (module MountingHole:MountingHole_3.5mm (layer F.Cu)
+    (at 18.288 18.288)
+    (descr "Mounting Hole 3.5mm, no annular")
+    (tags "mounting hole 3.5mm no annular")
+    (attr virtual)
+    (fp_text reference REF** (at 0 -4.5) (layer F.SilkS)
+      (effects (font (size 1 1) (thickness 0.15)))
+    )
+    (fp_text value MountingHole_3.5mm (at 0 4.5) (layer F.Fab)
+      (effects (font (size 1 1) (thickness 0.15)))
+    )
+    (fp_circle (center 0 0) (end 3.75 0) (layer F.CrtYd) (width 0.05))
+    (fp_circle (center 0 0) (end 3.5 0) (layer Cmts.User) (width 0.15))
+    (fp_text user %R (at 0.3 0) (layer F.Fab)
+      (effects (font (size 1 1) (thickness 0.15)))
+    )
+    (pad 1 np_thru_hole circle (at 0 0) (size 3.5 3.5) (drill 3.5) (layers *.Cu *.Mask))
+  )
   (module Capacitor_THT:C_Rect_L7.0mm_W2.5mm_P5.00mm (layer F.Cu)
