File: Diode VCF -  Hyperreal/Diode VCF -  Hyperreal.sch (KiCad schematic (older format))
At the start: 65 parts, among them J1 CV_In, J2 Sig_In, J3 Sig_Out, J4 Conn_01x02_Female, J5 Conn_01x02_Female, J6 Conn_01x02_Female, Q1 BC109, Q2 BC109, Q3 BC109, Q4 BC109, U1 TL074

Commit message: hii
Parts:
- added J7: Freq_Off, Connector_Wire:SolderWirePad_1x01_Drill1mm, symbol Connector:Conn_01x01_Female
- added R24: 1k, Resistor_THT:R_Axial_DIN0207_L6.3mm_D2.5mm_P7.62mm_Horizontal, symbol Device:R_US
- C1: value 4k7 -> 4u7; footprint (none) -> Capacitor_THT:CP_Radial_D5.0mm_P2.0mm_Bigger_Holes
- C10, C9: value C_Small -> 100n; footprint (none) -> Capacitor_THT:C_Rect_L7.0mm_W2.5mm_P5.00mm
- C11, C12: value CP1 -> 10u; footprint (none) -> Capacitor_THT:CP_Radial_D5.0mm_P2.0mm_Bigger_Holes
- C2, C3, C4, C5, C6, C7: footprint (none) -> Capacitor_THT:C_Rect_L7.0mm_W2.5mm_P5.00mm
- C8: footprint (none) -> Capacitor_THT:CP_Radial_D5.0mm_P2.0mm_Bigger_Holes
- D1, D10, D11, D12, D13, D14, D15, D16, D2, D3, D4, D5, D6, D7, D8, D9: footprint (none) -> Diode_THT:D_T-1_P5.08mm_Horizontal
- J1, J2, J3: footprint (none) -> Connector_Wire:SolderWirePad_1x01_Drill1mm
- J4: value Conn_01x02_Female -> +12V; footprint (none) -> Connector_Wire:SolderWirePad_1x02_P3.81mm_Drill1mm
- J5: value Conn_01x02_Female -> GND; footprint (none) -> Connector_Wire:SolderWirePad_1x02_P3.81mm_Drill1mm
- J6: value Conn_01x02_Female -> -12V; footprint (none) -> Connector_Wire:SolderWirePad_1x02_P3.81mm_Drill1mm
- R1, R10, R11, R12, R13, R14, R15, R16, R17, R18, R19, R2, R20, R21, R22, R23, R3, R4, R5, R6, R7, R8, R9: footprint (none) -> Resistor_THT:R_Axial_DIN0207_L6.3mm_D2.5mm_P7.62mm_Horizontal
- RV2: footprint (none) -> Potentiometer_THT:Potentiometer_Runtron_RM-065_Vertical
- U1: footprint (none) -> Package_DIP:DIP-14_W7.62mm_Socket
Connections:
- net Earth: no longer U1.12 (+)
- net at RV3.2: now also U1.12 (+); no longer J3.1 (Pin_1)
- net at R2.2, RV1.2: now also J7.1 (Pin_1)
- net at U1.13 (-), U1.14: now also R24.2
- new net: J3.1 (Pin_1), R24.1
Other:
- moved on the sheet: J3, RV1, U1D
