File: Diode VCF -  Hyperreal/Diode VCF -  Hyperreal.kicad_pcb (KiCad board)
At the start: 2 copper layers, 59 x 78 mm, 71 parts, among them J1 CV_In, J2 Sig_In, J3 Sig_Out, J4 +12V, J5 GND, J6 -12V, J7 Freq_Off, Q1 BC109, Q2 BC109, Q3 BC109, Q4 BC109, U1 TL074

Commit message: wuw
Other:
- board text added: "+12V"
- board text added: "-12V"
- board text added: "CV"
- board text added: "Freq"
- board text added: "GND"
- board text added: "Out"
- board text added: "Sig_In"
- board text added: "TL074"
