File: Diode VCF - Synthi Clone/Diode VCF - Synthi Clone.sch (KiCad schematic (older format))
At the start: 14 parts

Commit message: uwu
Parts:
- removed U?: CA3096, symbol modular_synth:CA3096
- added C?: 16u, symbol Device:CP1_Small
- added C?: CP1_Small, symbol Device:CP1_Small
- added C? (x4): 100n, symbol Device:C_Small
- added D? (x14): 1N914, symbol Device:D_Small
- added J?: Out, symbol Connector:Conn_01x01_Female
- added J?: In1, symbol Connector:Conn_01x01_Female
- added J?: In2, symbol Connector:Conn_01x01_Female
- added Q? (x2): BC557, Package_TO_SOT_THT:TO-92_Inline, symbol Transistor_BJT:BC557
- added Q? (x3): BC547, Package_TO_SOT_THT:TO-92_Inline, symbol Transistor_BJT:BC547
- added R? (x2): 10k, symbol Device:R_US
- added R?: 1k, symbol Device:R_US
- added R?: 100k, symbol Device:R_US
- added R? (x2): R_US, symbol Device:R_US
- added R?: 8k2, symbol Device:R_US
- added R? (x2): 2k2, symbol Device:R_US
- added U?: TL074, symbol Amplifier_Operational:TL074
Connections:
- net labels added: -9V, Earth
- wire segments 61 -> 95
Other:
- moved on the sheet: R?, U?A, U?E
