File: EchoFXXX_MFOS/EchoFXXX_MFOS.sch (KiCad schematic (older format))
At the start: 101 parts, among them J1 +5, J10 Conn_01x10_Female, J11 +12v, J12 GND, J13 -12v, J14 Out, J15 Dry1, J16 Dry2, J2 -5, J3 Fdbk_CV, J4 Fdbk, J5 In, J6 Wet_CV, J7 Wet, J8 Del_Time_CV, J9 Del_Time_Adj, Q1 2N3906, Q2 2N3906, Q3 2N3904, Q4 2N3904, U1 L7805, U2 PT2399, U3 TL074, U4 TL074, U5 LM13700

Commit message: wuw
Other:
- note added: "NP"
- note added: "NP\n"
Changed lines of the file:
@@
 	1    0    0    -1
 $EndComp
+Text Notes 9550 2400 0    50   ~ 0
+NP
+Text Notes 3950 800  0    50   ~ 0
+NP
+Text Notes 3900 1600 0    50   ~ 0
+NP
+Text Notes 7800 1850 0    50   ~ 0
+NP
+Text Notes 1350 3750 0    50   ~ 0
+NP\n
+Text Notes 8950 1850 0    50   ~ 0
+NP
 $EndSCHEMATC
