File: Gated Comparator - Serge/Gated Comparator - Serge.sch (KiCad schematic (older format))
At the start: 114 parts

Commit message: uwu
Parts:
- removed R? (x2): 10k, symbol Device:R_US
- removed RV?: 10k, symbol Device:R_POT_US
- added J30: Sens_Pot, Connector_Wire:SolderWirePad_1x01_Drill1mm, symbol Connector:Conn_01x01_Female
- added J31: Man_Loop, Connector_Wire:SolderWirePad_1x01_Drill1mm, symbol Connector:Conn_01x01_Female
- added R16: 15k, Resistor_THT:R_Axial_DIN0207_L6.3mm_D2.5mm_P7.62mm_Horizontal, symbol Device:R_US
- C1, C2: renamed from C?; footprint (none) -> Capacitor_THT:C_Rect_L7.0mm_W2.5mm_P5.00mm
- D1, D2: renamed from D?; footprint (none) -> Diode_THT:D_T-1_P5.08mm_Horizontal
- J1, J15, J18, J2, J3, J4, J5, J6, J7, J8: renamed from J?; footprint (none) -> Connector_Wire:SolderWirePad_1x01_Drill1mm
- J10: renamed from J?; value L1 -> L3; footprint (none) -> Connector_Wire:SolderWirePad_1x01_Drill1mm
- J11: renamed from J?; value L1 -> L6; footprint (none) -> Connector_Wire:SolderWirePad_1x01_Drill1mm
- J12: renamed from J?; value O1 -> OC; footprint (none) -> Connector_Wire:SolderWirePad_1x01_Drill1mm
- J13: renamed from J?; value O1 -> O3; footprint (none) -> Connector_Wire:SolderWirePad_1x01_Drill1mm
- J14: renamed from J?; value O1 -> O6; footprint (none) -> Connector_Wire:SolderWirePad_1x01_Drill1mm
- J16: renamed from J?; value L1 -> L4; footprint (none) -> Connector_Wire:SolderWirePad_1x01_Drill1mm
- J17: renamed from J?; value L1 -> L7; footprint (none) -> Connector_Wire:SolderWirePad_1x01_Drill1mm
- J19: renamed from J?; value O1 -> O4; footprint (none) -> Connector_Wire:SolderWirePad_1x01_Drill1mm
- J20: renamed from J?; value O1 -> O7; footprint (none) -> Connector_Wire:SolderWirePad_1x01_Drill1mm
- J21: renamed from J?; value L1 -> L2; footprint (none) -> Connector_Wire:SolderWirePad_1x01_Drill1mm
- J22: renamed from J?; value L1 -> L5; footprint (none) -> Connector_Wire:SolderWirePad_1x01_Drill1mm
- J23: renamed from J?; value L1 -> L8; footprint (none) -> Connector_Wire:SolderWirePad_1x01_Drill1mm
- J24: renamed from J?; value O1 -> O2; footprint (none) -> Connector_Wire:SolderWirePad_1x01_Drill1mm
- J25: renamed from J?; value O1 -> O5; footprint (none) -> Connector_Wire:SolderWirePad_1x01_Drill1mm
- J26: renamed from J?; value O1 -> O8; footprint (none) -> Connector_Wire:SolderWirePad_1x01_Drill1mm
- J9: renamed from J?; value L1 -> LC; footprint (none) -> Connector_Wire:SolderWirePad_1x01_Drill1mm
- Q1, Q10, Q2, Q3, Q4, Q5, Q6, Q7, Q8, Q9: renamed from Q?; footprint Package_TO_SOT_THT:TO-92_Inline -> Package_TO_SOT_THT:TO-92_Inline_Wide
- R1, R10, R11, R12, R13, R14, R15, R18, R19, R2, R20, R21, R22, R23, R24, R25, R26, R27, R28, R29, R3, R30, R31, R32, R33, R34, R35, R36, R37, R38, R39, R4, R40, R41, R42, R43, R44, R45, R46, R47, R48, R49, R5, R50, R51, R52, R53, R54, R55, R56, R57, R58, R59, R6, R60, R61, R62, R7, R8, R9: renamed from R?; footprint (none) -> Resistor_THT:R_Axial_DIN0207_L6.3mm_D2.5mm_P7.62mm_Horizontal
- U1, U2, U3: renamed from U?; footprint (none) -> Package_DIP:DIP-8_W7.62mm_Socket
- U4: renamed from U?; footprint (none) -> Package_DIP:DIP-16_W7.62mm_Socket
Connections:
- net at C1.1, R1.1, R4.2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: now also R16.1
- net at R15.2: now also J30.1 (Pin_1)
- new net: J31.1 (Pin_1), R16.2

Commit message: wuw
Other:
- note added: "LOTS OF\nTHESE\n200Ks\nSHOULD \nBE 100k\n"
Changed lines of the file:
@@
 Wire Wire Line
 	1900 1500 2100 1500
+Text Notes 7350 2200 0    50   ~ 0
+LOTS OF\nTHESE\n200Ks\nSHOULD \nBE 100k\n
 $EndSCHEMATC
