File: Smooth and Stepped Generator - CGS/Smooth and Stepped Generator - CGS.sch (KiCad schematic (older format))
At the start: 112 parts, among them J1 IN_A, J10 LA_A, J11 LK_A, J12 OUT_B, J13 CYCLE_B, J14 CYCLE_A, J15 COUPLER, J16 CA, J17 CK, J18 RD_OUT, J19 +12V_Conn, J2 IN_B, J20 GND_Conn, J21 -12V_Conn, J22 RATE_A, J23 RATE_B, J3 VC_A, J4 VC_B, J5 HOLD_A, J6 SAMPLE, J7 LA_B, J8 LK_B, J9 OUT_A, Q1 2N3906, Q2 2N3906, Q3 Q_NJFET_GDS, Q4 Q_NJFET_GDS, U1 LM3900, U2 CA3080, U3 CA3080, U4 TL072, U5 TL072, U7 LM741, U8 LM3900

Commit message: ssg work
Parts:
- D8: footprint Connector_Wire:SolderWirePad_1x01_Drill1mm -> Diode_THT:D_T-1_P5.08mm_Horizontal
- J18: footprint Connector_Wire:SolderWirePad_1x02_P3.81mm_Drill1mm -> Connector_Wire:SolderWirePad_1x01_Drill1mm
Connections:
- net at J3.1 (Pin_1): now also R13.2, R7.1, RV3.2; no longer RV3.1
- net at J4.1 (Pin_1): now also R14.2, R8.1, RV4.2; no longer RV4.1
Other:
- moved on the sheet: J3, J4
Changed lines of the file:
@@
 EESchema Schematic File Version 4
+LIBS:Smooth and Stepped Generator - CGS-cache
 EELAYER 29 0
 EELAYER END
@@
 L Connector:Conn_01x01_Female J3
 U 1 1 606CE775
-P 700 2250
-F 0 "J3" H 592 2025 50  0000 C CNN
-F 1 "VC_A" H 592 2116 50  0000 C CNN
-F 2 "Connector_Wire:SolderWirePad_1x01_Drill1mm" H 700 2250 50  0001 C CNN
-F 3 "~" H 700 2250 50  0001 C CNN
-	1    700  2250
-	-1   0    0    1
+P 1200 2250
+F 0 "J3" V 1350 2250 50  0000 C CNN
+F 1 "VC_A" V 1250 2250 50  0000 C CNN
+F 2 "Connector_Wire:SolderWirePad_1x01_Drill1mm" H 1200 2250 50  0001 C CNN
+F 3 "~" H 1200 2250 50  0001 C CNN
+	1    1200 2250
+	0    -1   -1   0
 $EndComp
 $Comp
@@
 P 1450 2450
 F 0 "R13" V 1245 2450 50  0000 C CNN
-F 1 "2M7" V 1336 2450 50  0000 C CNN
+F 1 "2M7" V 1350 2450 50  0000 C CNN
 F 2 "Resistor_THT:R_Axial_DIN0207_L6.3mm_D2.5mm_P7.62mm_Horizontal" V 1490 2440 50  0001 C CNN
 F 3 "~" H 1450 2450 50  0001 C CNN
@@
 L Connector:Conn_01x01_Female J4
 U 1 1 6074F552
-P 700 5850
-F 0 "J4" H 592 5625 50  0000 C CNN
-F 1 "VC_B" H 592 5716 50  0000 C CNN
-F 2 "Connector_Wire:SolderWirePad_1x01_Drill1mm" H 700 5850 50  0001 C CNN
-F 3 "~" H 700 5850 50  0001 C CNN
-	1    700  5850
-	-1   0    0    1
+P 1200 5850
+F 0 "J4" V 1350 5850 50  0000 C CNN
+F 1 "VC_B" V 1250 5850 50  0000 C CNN
+F 2 "Connector_Wire:SolderWirePad_1x01_Drill1mm" H 1200 5850 50  0001 C CNN
+F 3 "~" H 1200 5850 50  0001 C CNN
+	1    1200 5850
+	0    -1   -1   0
 $EndComp
 $Comp
@@
 F 0 "D8" V 8700 3350 50  0000 L CNN
 F 1 "D" V 8800 3350 50  0000 L CNN
-F 2 "Connector_Wire:SolderWirePad_1x01_Drill1mm" H 8750 3500 50  0001 C CNN
+F 2 "Diode_THT:D_T-1_P5.08mm_Horizontal" H 8750 3500 50  0001 C CNN
 F 3 "~" H 8750 3500 50  0001 C CNN
 	1    8750 3500
@@
 F 0 "J18" H 9578 4126 50  0000 L CNN
 F 1 "RD_OUT" H 9578 4035 50  0000 L CNN
-F 2 "Connector_Wire:SolderWirePad_1x02_P3.81mm_Drill1mm" H 9550 4100 50  0001 C CNN
+F 2 "Connector_Wire:SolderWirePad_1x01_Drill1mm" H 9550 4100 50  0001 C CNN
 F 3 "~" H 9550 4100 50  0001 C CNN
 	1    9550 4100

Commit message: wuw
Other:
- note added: "should be +12"
Changed lines of the file:
@@
 $EndComp
 Connection ~ 1100 7600
+Text Notes 7400 4850 0    50   ~ 0
+should be +12
 $EndSCHEMATC
