File: Wavefolder - Yusynth/Wavefolder - Yusynth.kicad_pcb (KiCad board)
At the start: 2 copper layers, 90 parts, among them J1 In, J2 +12v, J3 GND, J4 -12v, J5 CV, J6 Out, J7 Range, J8 Shape3, J9 Shape2, Q1 BC547, Q2 BC547, Q3 BC547, U1 TL072, U2 TL074

Commit message: uwu
Other:
- board outline added: 77 x 65 mm
Changed lines of the file:
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@@
   (general
     (thickness 1.6)
-    (drawings 4)
+    (drawings 8)
     (tracks 395)
     (zones 0)
@@
     (44 Edge.Cuts user)
     (45 Margin user)
-    (46 B.CrtYd user)
-    (47 F.CrtYd user)
+    (46 B.CrtYd user hide)
+    (47 F.CrtYd user hide)
     (48 B.Fab user)
     (49 F.Fab user)
@@
     )
   )
+  (gr_line (start 89 12) (end 12 12) (layer Edge.Cuts) (width 0.05))
+  (gr_line (start 89 77) (end 89 12) (layer Edge.Cuts) (width 0.05))
+  (gr_line (start 12 77) (end 89 77) (layer Edge.Cuts) (width 0.05))
+  (gr_line (start 12 12) (end 12 77) (layer Edge.Cuts) (width 0.05))
   (gr_line (start 89 12) (end 12 12) (layer F.SilkS) (width 0.12))
   (gr_line (start 89 77) (end 89 12) (layer F.SilkS) (width 0.12))
